File: REX1_bkw.sch (KiCad schematic (older format))
At the start: 10 parts, among them J1 Molex_DIP28_edge_contacts, J2 JTAG, J3 PRG, U1 XCR3064XL-10VQ44, U2 29F800, U3 LP2980

Commit message: reduce X & Y for 3d printing variability
Parts:
- J1: footprint 000_LOCAL:pcb2molex8878 -> 000_LOCAL:pcb2molex8878_chamfer
Changed lines of the file:
@@
 Title "REX1 bkw"
 Date "2019-06-29"
-Rev "4"
+Rev "12"
 Comp ""
 Comment1 "Original: Steven Adolph"
@@
 F 0 "J1" H 2720 5080 50  0000 C CNN
 F 1 "Molex_DIP28_edge_contacts" H 2700 6720 50  0000 C CNN
-F 2 "000_LOCAL:pcb2molex8878" H 2262 4998 60  0001 L CNN
+F 2 "000_LOCAL:pcb2molex8878_chamfer" H 2262 4998 60  0001 L CNN
 F 3 "" H 3000 6160 60  0001 L CNN
 	1    2800 5860
