File: REX1_NEC_bkw.kicad_pcb (KiCad board)
At the start: 2 copper layers, 16.4 x 34.2 mm, 9 parts, among them J1 DIP28_NEC_MAIN_ROM, J2 JTAG, J3 PRG, U1 XCR3064XL-10VQ44, U2 29F800, U3 LP2980

Commit message: silkscreen
Routing:
- net /TP1: track 14.3 -> 12.0 mm
- net /+5: track 58.7 -> 56.4 mm
- net /A11: track 17.0 -> 18.0 mm
- net /LVA3: track 7.41 -> 6.74 mm
Other:
- board text added: "1"
- board text added: "BKW_N2"
- board text removed: "BKW_12"
