File: REX_bkw.sch (KiCad schematic (older format))
At the start: 10 parts, among them J1 Molex_DIP28_edge_contacts, J2 JTAG, J3 PRG, U1 XCR3064XL-10VQ44, U2 29F800, U3 LP2980

Commit message: names
Parts:
- U1: symbol 000_LOCAL:XCR3064XL-10VQ44 -> 000_LOCAL:XCR3064-VQ44_
- U2: symbol 000_LOCAL:29F800 -> 000_LOCAL:29F800_
Connections:
- wire segments 152 -> 153
Changed lines of the file:
@@
 encoding utf-8
 Sheet 1 1
-Title "REX1 bkw"
+Title "REX bkw"
 Date "2019-06-29"
 Rev "12"
@@
 Wire Wire Line
 	8430 4090 8430 4590
-Text Label 8430 4390 1    50   ~ 0
+Text Label 8430 4590 1    50   ~ 0
 GND
 Wire Wire Line
@@
 Text Label 4730 3790 0    50   ~ 0
 ALE
-Text Label 8130 4290 1    50   ~ 0
+Text Label 8130 4590 1    50   ~ 0
 ALE
 Text Label 3420 5910 2    50   ~ 0
@@
 Wire Wire Line
 	7930 4090 7930 4590
-Text Label 7930 4390 1    50   ~ 0
+Text Label 7930 4590 1    50   ~ 0
 +3V3
 Wire Wire Line
@@
 1 uf
 Connection ~ 13030 8190
-Text Label 8230 4190 1    50   ~ 0
+Text Label 8230 4590 1    50   ~ 0
 ~RESET
 Text Label 3420 5310 2    50   ~ 0
@@
 $EndComp
 $Comp
-L 000_LOCAL:XCR3064XL-10VQ44 U1
+L 000_LOCAL:XCR3064-VQ44_ U1
 U 1 1 5D2858A9
 P 8530 5290
@@
 $EndComp
 $Comp
-L 000_LOCAL:29F800 U2
+L 000_LOCAL:29F800_ U2
 U 1 1 5D294874
 P 13730 5190
@@
 Wire Bus Line
 	10800 8190 13030 8190
+Wire Wire Line
+	12930 6590 13030 6590
+Wire Wire Line
+	13030 6590 13530 6590
 Wire Bus Line
 	4630 7060 4630 8190
@@
 Wire Bus Line
 	5630 8290 16130 8290
-Wire Wire Line
-	12930 6590 13530 6590
 Wire Bus Line
 	16130 4390 16130 8290
@@
 	15630 5590 15630 8190
 Wire Bus Line
+	13030 4790 13030 6590
+Wire Bus Line
+	13030 6590 13030 8190
+Wire Bus Line
 	4630 2790 4630 7060
 Wire Bus Line
 	3520 5110 3520 7060
-Wire Bus Line
-	13030 4790 13030 8190
 $EndSCHEMATC

Commit message: v13
Parts:
- added NT1, NT2, NT3, NT4, NT5, NT6: Net-Tie_2, 000_LOCAL:Net_Tie_2_0.18mm, symbol Device:Net-Tie_2
- C1: footprint Capacitors_SMD:C_0805 -> 000_LOCAL:C_0805; symbol Device:C -> 000_LOCAL:C
- J1: footprint 000_LOCAL:pcb2molex8878_chamfer -> 000_LOCAL:pcb2molex8878
- R1: footprint Resistors_SMD:R_0805 -> 000_LOCAL:R_0805; symbol Device:R -> 000_LOCAL:R
Connections:
- net labels added: D0, D1, D2, D3, D4, D5, D6, D7, ~BYTE
- net labels removed: AD0, AD1, AD2, AD3, AD4, AD5, AD6, AD7
- wire segments 153 -> 160
- no-connect marks 0 -> 13
Changed lines of the file:
@@
 	15230 6990 14730 6990
 Wire Wire Line
-	14730 5290 15130 5290
-Wire Wire Line
-	15130 5290 15130 5390
-Wire Wire Line
 	15330 5390 15230 5390
-Wire Wire Line
-	15230 5390 15130 5390
-Wire Wire Line
-	15130 5390 14730 5390
 Wire Wire Line
 	15230 5690 15230 5390
@@
 Connection ~ 15230 6590
 Connection ~ 15230 6790
-Connection ~ 15130 5390
 Connection ~ 15230 5690
 Connection ~ 15230 5390
-Text Label 15130 5290 0    50   ~ 0
-GND
+Text Label 14730 5290 0    50   ~ 0
+~BYTE
 Wire Wire Line
 	8430 4090 8430 4590
@@
 	15530 6690 14730 6690
 Text Label 15530 6690 2    50   ~ 0
-AD2
+D2
 Wire Wire Line
 	10700 5390 9230 5390
 Text Label 10700 5390 2    50   ~ 0
-AD2
+D2
 Wire Wire Line
 	15530 6890 14730 6890
 Text Label 15530 6890 2    50   ~ 0
-AD1
+D1
 Wire Wire Line
 	10700 5290 9230 5290
 Text Label 10700 5290 2    50   ~ 0
-AD1
+D1
 Text Label 3490 3120 2    50   ~ 0
-AD1
+D1
 Wire Wire Line
 	15530 7090 14730 7090
 Text Label 15530 7090 2    50   ~ 0
-AD0
+D0
 Wire Wire Line
 	10700 5190 9230 5190
 Text Label 10700 5190 2    50   ~ 0
-AD0
+D0
 Wire Wire Line
 	15530 6490 14730 6490
 Text Label 15530 6490 2    50   ~ 0
-AD3
+D3
 Wire Wire Line
 	10700 5490 9230 5490
 Text Label 10700 5490 2    50   ~ 0
-AD3
+D3
 Wire Wire Line
 	15530 6190 14730 6190
 Text Label 15530 6190 2    50   ~ 0
-AD4
+D4
 Wire Wire Line
 	10700 5690 9230 5690
 Text Label 10700 5690 2    50   ~ 0
-AD4
+D4
 Wire Wire Line
 	15530 5990 14730 5990
 Text Label 15530 5990 2    50   ~ 0
-AD5
+D5
 Wire Wire Line
 	10700 5790 9230 5790
 Text Label 10700 5790 2    50   ~ 0
-AD5
+D5
 Wire Wire Line
 	15530 5790 14730 5790
 Text Label 15530 5790 2    50   ~ 0
-AD6
+D6
 Wire Wire Line
 	10700 5890 9230 5890
 Text Label 10700 5890 2    50   ~ 0
-AD6
+D6
 Wire Wire Line
 	15530 5590 14730 5590
 Text Label 15530 5590 2    50   ~ 0
-AD7
+D7
 Wire Wire Line
 	10700 5990 9230 5990
 Text Label 10700 5990 2    50   ~ 0
-AD7
+D7
 Text Label 12930 6590 0    50   ~ 0
 RY_BY
@@
 Text Label 1130 7160 0    50   ~ 0
 +5
-Text Label 4730 2790 0    50   ~ 0
+Text Label 4730 2890 0    50   ~ 0
 +5
 Text Label 3420 5210 2    50   ~ 0
@@
 	3490 4260 3590 4160
 Entry Wire Line
-	4630 2890 4730 2790
+	4630 2900 4730 3000
 Entry Wire Line
 	4630 3490 4730 3590
@@
 	16030 7190 16130 7090
 $Comp
-L Device:C C1
+L 000_LOCAL:C C1
 U 1 1 327B8ADF
 P 3830 8940
 F 0 "C1" H 3950 8910 59  0000 L BNN
 F 1 "C-USC0805" H 3950 8810 59  0001 L BNN
-F 2 "Capacitors_SMD:C_0805" H 3830 8940 50  0001 C CNN
+F 2 "000_LOCAL:C_0805" H 3830 8940 50  0001 C CNN
 F 3 "" H 3830 8940 50  0001 C CNN
 	1    3830 8940
@@
 $EndComp
 $Comp
-L Device:R R1
+L 000_LOCAL:R R1
 U 1 1 2604F989
 P 3890 7870
 F 0 "R1" V 4010 7820 59  0000 L BNN
 F 1 "10k" H 3740 7740 59  0001 L BNN
-F 2 "Resistors_SMD:R_0805" H 3890 7870 50  0001 C CNN
+F 2 "000_LOCAL:R_0805" H 3890 7870 50  0001 C CNN
 F 3 "" H 3890 7870 50  0001 C CNN
 	1    3890 7870
@@
 	2430 8490 2690 8490
 Connection ~ 1130 8490
-Wire Wire Line
-	8230 2790 8230 4590
 Entry Wire Line
 	12730 4390 12830 4490
@@
 	8630 4490 12730 4490
 Wire Wire Line
-	4730 2790 8230 2790
+	4730 2890 4800 2890
 Text Label 3490 4260 2    50   ~ 0
 PORT_EN
@@
 	3490 3020 3590 2920
 Text Label 3490 3020 2    50   ~ 0
-AD6
+D6
 Wire Wire Line
 	7630 7290 6530 7290
@@
 TMS
 Wire Wire Line
-	2530 3320 3490 3320
-Wire Wire Line
-	2530 3220 3490 3220
-Wire Wire Line
-	2530 3120 3490 3120
-Wire Wire Line
-	2530 3020 3490 3020
+	2530 3320 2900 3320
+Wire Wire Line
+	2530 3220 2900 3220
+Wire Wire Line
+	2530 3120 2900 3120
+Wire Wire Line
+	2530 3020 2900 3020
 Text Label 2530 3220 0    50   ~ 0
 TDI
@@
 	3420 5910 3520 5810
 Text Label 2080 6410 0    50   ~ 0
-AD2
+D2
 Entry Wire Line
 	3420 5810 3520 5710
 Text Label 2080 6310 0    50   ~ 0
-AD1
+D1
 Entry Wire Line
 	3420 5710 3520 5610
 Text Label 2080 6210 0    50   ~ 0
-AD0
+D0
 Entry Wire Line
 	1980 5210 2080 5310
@@
 A10
 Text Label 3420 6510 2    50   ~ 0
-AD3
+D3
 Text Label 3420 6410 2    50   ~ 0
-AD4
+D4
 Text Label 3420 6310 2    50   ~ 0
-AD5
+D5
 Text Label 3420 6210 2    50   ~ 0
-AD6
+D6
 Text Label 3420 6110 2    50   ~ 0
-AD7
+D7
 Entry Wire Line
 	3420 6410 3520 6310
@@
 F 0 "J1" H 2720 5080 50  0000 C CNN
 F 1 "Molex_DIP28_edge_contacts" H 2700 6720 50  0000 C CNN
-F 2 "000_LOCAL:pcb2molex8878_chamfer" H 2262 4998 60  0001 L CNN
+F 2 "000_LOCAL:pcb2molex8878" H 2262 4998 60  0001 L CNN
 F 3 "" H 3000 6160 60  0001 L CNN
 	1    2800 5860
@@
 Wire Bus Line
 	10800 8190 13030 8190
-Wire Wire Line
-	12930 6590 13030 6590
-Wire Wire Line
-	13030 6590 13530 6590
+Text Label 8330 4590 1    50   ~ 0
+~RD
+$Comp
+L Device:Net-Tie_2 NT1
+U 1 1 5FBB145C
+P 4900 2890
+F 0 "NT1" H 4900 3130 50  0001 C CNN
+F 1 "Net-Tie_2" H 4900 3030 50  0001 C CNN
+F 2 "000_LOCAL:Net_Tie_2_0.18mm" H 4900 2890 50  0001 C CNN
+F 3 "~" H 4900 2890 50  0001 C CNN
+	1    4900 2890
+	1    0    0    -1
+$EndComp
+Entry Wire Line
+	4630 3100 4730 3200
+Text Label 4730 3200 0    50   ~ 0
+~RESET
+Entry Wire Line
+	4630 2790 4730 2890
+Text Label 4730 3000 0    50   ~ 0
+~RESET
+Wire Wire Line
+	4730 3000 5000 3000
+Wire Wire Line
+	5000 3000 5000 2890
+Wire Wire Line
+	4730 3200 8230 3200
+Wire Wire Line
+	8230 3200 8230 4590
+NoConn ~ 7730 6790
+NoConn ~ 8330 6790
+NoConn ~ 8430 6790
+NoConn ~ 8530 6790
+NoConn ~ 7030 5890
+Wire Wire Line
+	14730 5390 15230 5390
+Connection ~ 4630 2790
+Text Label 4730 2600 0    50   ~ 0
+GND
+Entry Wire Line
+	4630 2610 4730 2710
+Wire Wire Line
+	4730 2600 4800 2600
+$Comp
+L Device:Net-Tie_2 NT2
+U 1 1 5FCB31BF
+P 4900 2600
+F 0 "NT2" H 4900 2840 50  0001 C CNN
+F 1 "Net-Tie_2" H 4900 2740 50  0001 C CNN
+F 2 "000_LOCAL:Net_Tie_2_0.18mm" H 4900 2600 50  0001 C CNN
+F 3 "~" H 4900 2600 50  0001 C CNN
+	1    4900 2600
+	1    0    0    -1
+$EndComp
+Entry Wire Line
+	4630 2500 4730 2600
+Text Label 4730 2710 0    50   ~ 0
+~BYTE
+Wire Wire Line
+	4730 2710 5000 2710
+Wire Wire Line
+	5000 2710 5000 2600
+Entry Wire Line
+	16030 5290 16130 5190
+Wire Wire Line
+	14730 5290 16030 5290
+Text Label 16030 5290 2    50   ~ 0
+~BYTE
+NoConn ~ 2400 6110
+NoConn ~ 2400 6010
+NoConn ~ 2400 5910
+NoConn ~ 2400 5810
+NoConn ~ 2400 5710
+NoConn ~ 2400 5610
+NoConn ~ 2400 5510
+NoConn ~ 2400 5410
+Wire Bus Line
+	4630 2500 4630 2790
 Wire Bus Line
 	4630 7060 4630 8190
@@
 Wire Bus Line
 	5630 8290 16130 8290
+Wire Wire Line
+	12930 6590 13530 6590
 Wire Bus Line
 	16130 4390 16130 8290
 Wire Bus Line
+	4630 8190 10800 8190
+Wire Bus Line
 	1980 5110 1980 7060
 Wire Bus Line
-	4630 8190 10800 8190
-Wire Bus Line
 	12830 4390 12830 6590
 Wire Bus Line
@@
 	15630 5590 15630 8190
 Wire Bus Line
-	13030 4790 13030 6590
-Wire Bus Line
-	13030 6590 13030 8190
-Wire Bus Line
 	4630 2790 4630 7060
 Wire Bus Line
 	3520 5110 3520 7060
+Wire Bus Line
+	13030 4790 13030 8190
+$Comp
+L Device:Net-Tie_2 NT3
+U 1 1 5FD83265
+P 3000 3020
+F 0 "NT3" H 3000 3050 50  0001 C CNN
+F 1 "Net-Tie_2" H 3000 2990 50  0001 C CNN
+F 2 "000_LOCAL:Net_Tie_2_0.18mm" H 3000 3020 50  0001 C CNN
+F 3 "~" H 3000 3020 50  0001 C CNN
+	1    3000 3020
+	1    0    0    -1
+$EndComp
+Wire Wire Line
+	3100 3020 3490 3020
+$Comp
+L Device:Net-Tie_2 NT4
+U 1 1 5FD846AF
+P 3000 3120
+F 0 "NT4" H 3000 3150 50  0001 C CNN
+F 1 "Net-Tie_2" H 3000 3090 50  0001 C CNN
+F 2 "000_LOCAL:Net_Tie_2_0.18mm" H 3000 3120 50  0001 C CNN
+F 3 "~" H 3000 3120 50  0001 C CNN
+	1    3000 3120
+	1    0    0    -1
+$EndComp
+Wire Wire Line
+	3100 3120 3490 3120
+$Comp
+L Device:Net-Tie_2 NT5
+U 1 1 5FD8498E
+P 3000 3220
+F 0 "NT5" H 3000 3250 50  0001 C CNN
+F 1 "Net-Tie_2" H 3000 3190 50  0001 C CNN
+F 2 "000_LOCAL:Net_Tie_2_0.18mm" H 3000 3220 50  0001 C CNN
+F 3 "~" H 3000 3220 50  0001 C CNN
+	1    3000 3220
+	1    0    0    -1
+$EndComp
+Wire Wire Line
+	3100 3220 3490 3220
+$Comp
+L Device:Net-Tie_2 NT6
+U 1 1 5FD84CB8
+P 3000 3320
+F 0 "NT6" H 3000 3350 50  0001 C CNN
+F 1 "Net-Tie_2" H 3000 3290 50  0001 C CNN
+F 2 "000_LOCAL:Net_Tie_2_0.18mm" H 3000 3320 50  0001 C CNN
+F 3 "~" H 3000 3320 50  0001 C CNN
+	1    3000 3320
+	1    0    0    -1
+$EndComp
+Wire Wire Line
+	3100 3320 3490 3320
 $EndSCHEMATC

Commit message: flip ram and reroute nec board, several other minor touches both boards
Parts:
- removed NT3, NT4, NT5, NT6: Net-Tie_2, 000_LOCAL:Net_Tie_2_0.18mm, symbol Device:Net-Tie_2
- R1: value 10k -> 47k
- U3: value LP2980 -> LP2980-3.3
Connections:
- net labels removed: TCK, TDI, TDO, TMS, VREF
- wire segments 160 -> 155
- no-connect marks 13 -> 18
Other:
- note added: "TCK"
- note added: "TDI"
- note added: "TDO"
- note added: "TMS"
- note added: "VREF"
- note removed: "10k"
- moved on the sheet: R1
Changed lines of the file:
@@
 encoding utf-8
 Sheet 1 1
-Title "REX bkw"
-Date "2019-06-29"
-Rev "12"
-Comp ""
-Comment1 "Original: Steven Adolph"
-Comment2 "Modified: Brian White"
+Title "REX Classic, BKW re-spin"
+Date "2020-11-30"
+Rev "13"
+Comp "Brian K. White - b.kenyon.w@gmail.com"
+Comment1 "Original design: Steven Adolph"
+Comment2 ""
 Comment3 ""
 Comment4 ""
@@
 Text Label 1130 7160 0    50   ~ 0
 +5
-Text Label 4730 2890 0    50   ~ 0
+Text Label 5200 8800 0    50   ~ 0
 +5
 Text Label 3420 5210 2    50   ~ 0
@@
 	15530 5790 15630 5690
 Entry Wire Line
-	15530 5590 15630 5690
+	15530 5590 15630 5490
 Entry Wire Line
 	15530 6290 15630 6190
@@
 	3490 4260 3590 4160
 Entry Wire Line
-	4630 2900 4730 3000
+	5100 8800 5200 8900
 Entry Wire Line
 	4630 3490 4730 3590
@@
 	8130 8290 8230 8190
 Entry Wire Line
-	5630 6290 5730 6190
+	5630 6090 5730 6190
 Entry Wire Line
 	16030 7390 16130 7290
@@
 L 000_LOCAL:R R1
 U 1 1 2604F989
-P 3890 7870
-F 0 "R1" V 4010 7820 59  0000 L BNN
-F 1 "10k" H 3740 7740 59  0001 L BNN
-F 2 "000_LOCAL:R_0805" H 3890 7870 50  0001 C CNN
-F 3 "" H 3890 7870 50  0001 C CNN
-	1    3890 7870
-	0    1    1    0
+P 5650 8600
+F 0 "R1" V 5770 8550 59  0000 L BNN
+F 1 "47k" V 5600 8520 59  0000 L BNN
+F 2 "000_LOCAL:R_0805" H 5650 8600 50  0001 C CNN
+F 3 "" H 5650 8600 50  0001 C CNN
+	1    5650 8600
+	0    -1   1    0
 $EndComp
 $Comp
@@
 Text Notes 13590 8090 0    60   ~ 0
 bottom boot\nAM29F800BB, MX29F800CB
-Text Notes 3810 7820 0    60   ~ 0
-10k
 Wire Wire Line
 	3830 9090 3830 9290
@@
 	8630 4490 12730 4490
 Wire Wire Line
-	4730 2890 4800 2890
+	5200 8800 5270 8800
 Text Label 3490 4260 2    50   ~ 0
 PORT_EN
@@
 	-1   0    0    -1
 $EndComp
-Text Label 2530 3320 0    50   ~ 0
-TMS
-Wire Wire Line
-	2530 3320 2900 3320
-Wire Wire Line
-	2530 3220 2900 3220
-Wire Wire Line
-	2530 3120 2900 3120
-Wire Wire Line
-	2530 3020 2900 3020
-Text Label 2530 3220 0    50   ~ 0
-TDI
-Text Label 2530 3120 0    50   ~ 0
-TDO
-Text Label 2530 3020 0    50   ~ 0
-TCK
-Text Label 2530 2920 0    50   ~ 0
-GND
-Text Label 2530 2820 0    50   ~ 0
-VREF
 Wire Wire Line
 	6520 7090 6630 7090
@@
 Wire Wire Line
 	1130 7160 1130 8490
-$Comp
-L 000_LOCAL:LP2980 U3
-U 1 1 5D30DD1C
-P 1830 8590
-F 0 "U3" H 1880 8320 59  0000 C CNN
-F 1 "LP2980" H 1950 8580 59  0000 C CNN
-F 2 "000_LOCAL:SOT-23-5" H 1830 8590 50  0001 C CNN
-F 3 "" H 1830 8590 50  0001 C CNN
-	1    1830 8590
-	1    0    0    -1
-$EndComp
-Entry Wire Line
-	4530 7870 4630 7770
-Wire Wire Line
-	4530 7870 4040 7870
+Entry Wire Line
+	5100 8500 5200 8600
 $Comp
 L power:GND #PWR0101
 U 1 1 5D3EDA7D
-P 3490 7870
-F 0 "#PWR0101" H 3490 7620 50  0001 C CNN
-F 1 "GND" V 3495 7742 50  0000 R CNN
-F 2 "" H 3490 7870 50  0001 C CNN
-F 3 "" H 3490 7870 50  0001 C CNN
-	1    3490 7870
-	0    1    1    0
-$EndComp
-Wire Wire Line
-	3490 7870 3740 7870
-Text Label 4530 7870 2    50   ~ 0
+P 5800 8600
+F 0 "#PWR0101" H 5800 8350 50  0001 C CNN
+F 1 "GND" V 5805 8472 50  0000 R CNN
+F 2 "" H 5800 8600 50  0001 C CNN
+F 3 "" H 5800 8600 50  0001 C CNN
+	1    5800 8600
+	0    -1   -1   0
+$EndComp
+Text Label 5200 8600 0    50   ~ 0
 PORT_EN
 $Comp
@@
 L Device:Net-Tie_2 NT1
 U 1 1 5FBB145C
-P 4900 2890
-F 0 "NT1" H 4900 3130 50  0001 C CNN
-F 1 "Net-Tie_2" H 4900 3030 50  0001 C CNN
-F 2 "000_LOCAL:Net_Tie_2_0.18mm" H 4900 2890 50  0001 C CNN
-F 3 "~" H 4900 2890 50  0001 C CNN
-	1    4900 2890
+P 5370 8800
+F 0 "NT1" H 5370 9040 50  0001 C CNN
+F 1 "Net-Tie_2" H 5370 8940 50  0001 C CNN
+F 2 "000_LOCAL:Net_Tie_2_0.18mm" H 5370 8800 50  0001 C CNN
+F 3 "~" H 5370 8800 50  0001 C CNN
+	1    5370 8800
 	1    0    0    -1
 $EndComp
@@
 ~RESET
 Entry Wire Line
-	4630 2790 4730 2890
-Text Label 4730 3000 0    50   ~ 0
+	5100 8700 5200 8800
+Text Label 5200 8900 0    50   ~ 0
 ~RESET
 Wire Wire Line
-	4730 3000 5000 3000
-Wire Wire Line
-	5000 3000 5000 2890
+	5200 8900 5470 8900
 Wire Wire Line
 	4730 3200 8230 3200
@@
 Wire Wire Line
 	14730 5390 15230 5390
-Connection ~ 4630 2790
-Text Label 4730 2600 0    50   ~ 0
+Text Label 5200 9100 0    50   ~ 0
 GND
 Entry Wire Line
-	4630 2610 4730 2710
-Wire Wire Line
-	4730 2600 4800 2600
+	5100 9100 5200 9200
+Wire Wire Line
+	5200 9100 5270 9100
 $Comp
 L Device:Net-Tie_2 NT2
 U 1 1 5FCB31BF
-P 4900 2600
-F 0 "NT2" H 4900 2840 50  0001 C CNN
-F 1 "Net-Tie_2" H 4900 2740 50  0001 C CNN
-F 2 "000_LOCAL:Net_Tie_2_0.18mm" H 4900 2600 50  0001 C CNN
-F 3 "~" H 4900 2600 50  0001 C CNN
-	1    4900 2600
+P 5370 9100
+F 0 "NT2" H 5370 9340 50  0001 C CNN
+F 1 "Net-Tie_2" H 5370 9240 50  0001 C CNN
+F 2 "000_LOCAL:Net_Tie_2_0.18mm" H 5370 9100 50  0001 C CNN
+F 3 "~" H 5370 9100 50  0001 C CNN
+	1    5370 9100
 	1    0    0    -1
 $EndComp
 Entry Wire Line
-	4630 2500 4730 2600
-Text Label 4730 2710 0    50   ~ 0
+	5100 9000 5200 9100
+Text Label 5200 9200 0    50   ~ 0
 ~BYTE
 Wire Wire Line
-	4730 2710 5000 2710
-Wire Wire Line
-	5000 2710 5000 2600
+	5200 9200 5470 9200
 Entry Wire Line
 	16030 5290 16130 5190
@@
 NoConn ~ 2400 5510
 NoConn ~ 2400 5410
-Wire Bus Line
-	4630 2500 4630 2790
+Wire Wire Line
+	2530 3020 3490 3020
+Wire Wire Line
+	2530 3120 3490 3120
+Wire Wire Line
+	2530 3220 3490 3220
+Wire Wire Line
+	2530 3320 3490 3320
+Text Notes 2530 3320 0    50   ~ 0
+TMS
+Text Notes 2530 3220 0    50   ~ 0
+TDI
+Text Notes 2530 3120 0    50   ~ 0
+TDO
+Text Notes 2530 3020 0    50   ~ 0
+TCK
+Text Notes 2530 2820 0    50   ~ 0
+VREF
+NoConn ~ 2430 8690
+Wire Bus Line
+	5630 6090 5630 8290
+NoConn ~ 13530 5990
+NoConn ~ 13530 6090
+NoConn ~ 13530 6390
+NoConn ~ 13530 6490
 Wire Bus Line
 	4630 7060 4630 8190
-Wire Bus Line
-	5630 6190 5630 8290
+Wire Wire Line
+	5200 8600 5500 8600
+Wire Wire Line
+	5470 8900 5470 8800
+Wire Wire Line
+	5470 9200 5470 9100
+$Comp
+L 000_LOCAL:LP2980 U3
+U 1 1 5D30DD1C
+P 1830 8590
+F 0 "U3" H 1880 8320 59  0000 C CNN
+F 1 "LP2980-3.3" H 1860 8860 59  0000 C CNN
+F 2 "000_LOCAL:SOT-23-5" H 1830 8590 50  0001 C CNN
+F 3 "" H 1830 8590 50  0001 C CNN
+	1    1830 8590
+	1    0    0    -1
+$EndComp
+Wire Bus Line
+	4630 8190 5100 8190
+Connection ~ 5100 8190
 Wire Bus Line
 	5630 8290 16130 8290
@@
 	16130 4390 16130 8290
 Wire Bus Line
-	4630 8190 10800 8190
+	5100 8190 5100 9100
 Wire Bus Line
 	1980 5110 1980 7060
 Wire Bus Line
-	12830 4390 12830 6590
+	5100 8190 10800 8190
+Wire Bus Line
+	12830 4390 12830 6490
 Wire Bus Line
 	3590 2790 3590 4160
@@
 	10800 5090 10800 8190
 Wire Bus Line
-	15630 5590 15630 8190
+	15630 5490 15630 8190
 Wire Bus Line
 	4630 2790 4630 7060
@@
 Wire Bus Line
 	13030 4790 13030 8190
-$Comp
-L Device:Net-Tie_2 NT3
-U 1 1 5FD83265
-P 3000 3020
-F 0 "NT3" H 3000 3050 50  0001 C CNN
-F 1 "Net-Tie_2" H 3000 2990 50  0001 C CNN
-F 2 "000_LOCAL:Net_Tie_2_0.18mm" H 3000 3020 50  0001 C CNN
-F 3 "~" H 3000 3020 50  0001 C CNN
-	1    3000 3020
-	1    0    0    -1
-$EndComp
-Wire Wire Line
-	3100 3020 3490 3020
-$Comp
-L Device:Net-Tie_2 NT4
-U 1 1 5FD846AF
-P 3000 3120
-F 0 "NT4" H 3000 3150 50  0001 C CNN
-F 1 "Net-Tie_2" H 3000 3090 50  0001 C CNN
-F 2 "000_LOCAL:Net_Tie_2_0.18mm" H 3000 3120 50  0001 C CNN
-F 3 "~" H 3000 3120 50  0001 C CNN
-	1    3000 3120
-	1    0    0    -1
-$EndComp
-Wire Wire Line
-	3100 3120 3490 3120
-$Comp
-L Device:Net-Tie_2 NT5
-U 1 1 5FD8498E
-P 3000 3220
-F 0 "NT5" H 3000 3250 50  0001 C CNN
-F 1 "Net-Tie_2" H 3000 3190 50  0001 C CNN
-F 2 "000_LOCAL:Net_Tie_2_0.18mm" H 3000 3220 50  0001 C CNN
-F 3 "~" H 3000 3220 50  0001 C CNN
-	1    3000 3220
-	1    0    0    -1
-$EndComp
-Wire Wire Line
-	3100 3220 3490 3220
-$Comp
-L Device:Net-Tie_2 NT6
-U 1 1 5FD84CB8
-P 3000 3320
-F 0 "NT6" H 3000 3350 50  0001 C CNN
-F 1 "Net-Tie_2" H 3000 3290 50  0001 C CNN
-F 2 "000_LOCAL:Net_Tie_2_0.18mm" H 3000 3320 50  0001 C CNN
-F 3 "~" H 3000 3320 50  0001 C CNN
-	1    3000 3320
-	1    0    0    -1
-$EndComp
-Wire Wire Line
-	3100 3320 3490 3320
 $EndSCHEMATC
