File: REX_Classic_bkw.sch (KiCad schematic (older format))
At the start: 12 parts, among them J1 Molex_DIP28_edge_contacts, J2 JTAG, J3 PRG, U1 XCR3064XL-10VQ44, U2 29F800, U3 LP2980-3.3

Commit message: Less expensive manufacturing tolerances. Rename to REX Classic.
Parts:
- J1: footprint 000_LOCAL:pcb2molex8878 -> 000_LOCAL:pcb2molex8878_contacts
Changed lines of the file:
@@
 F 0 "J1" H 2720 5080 50  0000 C CNN
 F 1 "Molex_DIP28_edge_contacts" H 2700 6720 50  0000 C CNN
-F 2 "000_LOCAL:pcb2molex8878" H 2262 4998 60  0001 L CNN
+F 2 "000_LOCAL:pcb2molex8878_contacts" H 2262 4998 60  0001 L CNN
 F 3 "" H 3000 6160 60  0001 L CNN
 	1    2800 5860

Commit message: min drill 0.3mm for PCBWAY, replace GND traces with zone fill
Parts:
- removed J1: Molex_DIP28_edge_contacts, 000_LOCAL:pcb2molex8878_contacts, symbol 000_LOCAL:Molex_DIP28_edge_contacts
- removed NT2: Net-Tie_2, 000_LOCAL:Net_Tie_2_0.18mm, symbol Device:Net-Tie_2
- added J1: TRS-80_Model_100_Option_ROM, 000_LOCAL:pcb2molex8878, symbol 000_LOCAL:TRS-80_Model_100_Option_ROM
Connections:
- net labels added: +5V, D1_TDO, D6_TCK, LVA19_TMS, LVA4_TDI, RY~BY, ~CE_MEM, ~CS_BUS, ~OE_BUS, ~OE_MEM
- net labels removed: +5, D1, D6, LVA19, LVA4, RY_BY, ~BYTE, ~CE, ~CS, ~OE, ~RD
- wire segments 155 -> 104
Other:
- note added: "3,4: jumper"
- note added: "GND"
- note removed: "3,4: short"
- moved on the sheet: C1, TP1, TP2

Commit message: rename pcb2molex8878 to Molex78805_PCB
Parts:
- J1: footprint 000_LOCAL:pcb2molex8878 -> 000_LOCAL:Molex78805_PCB
Changed lines of the file:
@@
 F 0 "J1" H 2750 6770 50  0000 C CNN
 F 1 "TRS-80_Model_100_Option_ROM" H 2750 6670 50  0000 C CNN
-F 2 "000_LOCAL:pcb2molex8878" H 2262 4998 60  0001 L CNN
+F 2 "000_LOCAL:Molex78805_PCB" H 2262 4998 60  0001 L CNN
 F 3 "" H 3000 6160 60  0001 L CNN
 	1    2800 5860
@@
 	16130 4390 16130 8290
 Wire Bus Line
-	5100 8190 10800 8190
-Wire Bus Line
 	1980 5210 1980 7060
 Wire Bus Line
@@
 	15630 5490 15630 8190
 Wire Bus Line
+	5100 8190 10800 8190
+Wire Bus Line
 	3590 2790 3590 4160

Commit message: upgrade board outline and carrier to v004
Parts:
- J1: footprint 000_LOCAL:Molex78805_PCB -> 000_LOCAL:Molex78802_PCB_28
Changed lines of the file:
@@
 Sheet 1 1
 Title "REX Classic, BKW re-spin"
-Date "2021-03-14"
-Rev "14"
+Date "2021-05-23"
+Rev "17"
 Comp "Brian K. White - b.kenyon.w@gmail.com"
 Comment1 "Original design: Steven Adolph"
@@
 F 0 "J1" H 2750 6770 50  0000 C CNN
 F 1 "TRS-80_Model_100_Option_ROM" H 2750 6670 50  0000 C CNN
-F 2 "000_LOCAL:Molex78805_PCB" H 2262 4998 60  0001 L CNN
+F 2 "000_LOCAL:Molex78802_PCB_28" H 2262 4998 60  0001 L CNN
 F 3 "" H 3000 6160 60  0001 L CNN
 	1    2800 5860
@@
 	12830 4390 12830 6490
 Wire Bus Line
+	5100 8190 10800 8190
+Wire Bus Line
 	15630 5490 15630 8190
 Wire Bus Line
-	5100 8190 10800 8190
-Wire Bus Line
 	3590 2790 3590 4160

Commit message: remove pointless busses from sch, minor silkscreen tweaks
Connections:
- net labels removed: TP1, TP2
- wire segments 104 -> 0
Other:
- moved on the sheet: C1, J2, J3, R1, TP1, TP2, U3

Commit message: clearances, remove pointless busses in schematic
Parts:
- removed U1: XCR3064XL-10VQ44, 000_LOCAL:QFP44, symbol 000_LOCAL:XCR3064-VQ44_
- removed U2: 29F800, 000_LOCAL:TSOP-48, symbol 000_LOCAL:29F800_
- added U1: XCR3064XL-VQ44, 000_LOCAL:VQFP44, symbol 000_LOCAL:XCR3064-VQ44
- added U2: 29F800, 000_LOCAL:TSOP-48, symbol 000_LOCAL:29F800
Connections:
- no-connect marks 18 -> 14
Other:
- moved on the sheet: C1, R1, U3
