File: REX_Sharp_DIP_bkw.kicad_sch (KiCad schematic)
At the start: 11 parts, among them J1 DIP28 legs 27C256, J2 JTAG, J3 PRG, U1 XCR3064-VQ44, U2 29F800BB, U3 LP2980-3.3

Commit message: kicad 7, 0.2mm tracks, 0.3x0.5mm vias, add caps on 3v3
Parts:
- removed J1: DIP28 legs 27C256, 000_LOCAL:DIP-28_600_pcb_shallow_notch, symbol 000_LOCAL:27C256
- removed J2: JTAG, 000_LOCAL:1x6_pcb_socket, symbol Connector:Conn_01x06_Female
- removed J3: PRG, 000_LOCAL:1x4_pcb_socket, symbol Connector:Conn_01x04_Female
- removed TP1: PINHD-1X1, 000_LOCAL:1x1_pin_h, symbol Connector:Conn_01x01_Male
- added J1: Option-ROM SOCKET, 000_LOCAL:DIP-28_600_pcb_shallow_notch, symbol 000_LOCAL:ROM_SOCKET
- added TP1: PORT_EN, 000_LOCAL:1x1_pin_h, symbol 000_LOCAL:TestPoint
- added TP2: 3V3/VREF, 000_LOCAL:1x1_pin_h, symbol 000_LOCAL:TestPoint
- C1, C3: value 1u -> 1uF
- C2: value 1u -> 100pF
- U1: value XCR3064-VQ44 -> XCR3032XL-VQ44
- U2: value 29F800BB -> 29F800 bottom boot
Connections:
- net TP1 is gone; now on net ~{BUS_CS}: U1.40 (CLC0/IN0)
- net +3V3: now also TP2.1; no longer C2.1
- net +5V: now also J1.28 (VCC); no longer U1.39 (CLK1/IN1)
- net A0: now also U1.6 (B14), J1.10 (A0); no longer U1.22 (C8)
- net A1: now also U1.5 (B13), J1.9 (A1); no longer U1.21 (C9)
- net A10: now also J1.21 (A10)
- net A11: now also J1.23 (A11)
- net A12: now also J1.2 (A12)
- net A13: now also J1.26 (A13)
- net A14: now also J1.27 (A14)
- net A16: now also U1.28 (A13); no longer U1.5 (B13)
- net A17: now also U1.33 (A7); no longer U1.2 (B9)
- net A18: now also U1.13 (D9); no longer U1.19 (C11)
- net A2: now also U1.11 (D4), J1.8 (A2); no longer U1.20 (C10)
- net A3: now also U1.10 (D3), J1.7 (A3); no longer U1.18 (C12)
- net A4: now also U1.2 (B9), J1.6 (A4); no longer U1.15 (D11)
- net A5: now also U1.3 (B10), J1.5 (A5); no longer U1.14 (D10)
- net A6: now also U1.44 (B2), J1.4 (A6); no longer U1.13 (D9)
- net A7: now also J1.3 (A7)
- net A9: now also J1.24 (A9)
- net D0: now also U1.8 (D1), J1.11 (D0); no longer U1.23 (C3)
- net D4: now also U1.30 (A10), J1.16 (D4); no longer U1.31 (A9)
- net D6: now also U1.25 (C1), J1.18 (D6); no longer U1.33 (A7)
- net D7: now also U1.23 (C3), J1.19 (D7); no longer U1.34 (A1)
- net GND: now also U2.10 (NC), U2.13 (NC), U2.14 (NC), U2.9 (NC(A19)), J1.14 (GND)
- net PORT_EN: now also TP1.1
- net RY/~{BY}: now also U1.15 (D11); no longer U1.6 (B14)
- net ~{BUS_CS}: now also J1.20 (~{CE}); no longer U1.37 (CLK3/IN3)
- net ~{BUS_OE}: now also C2.1, J1.22 (~{OE})
- net A15/TMS renamed A15
- net A15: now also U1.31 (A9); no longer U1.7 (D0/TMS)
- net A19/TCK renamed A19
- net A19: now also U1.14 (D10); no longer U1.26 (C0/TCK)
- net A8/TDI renamed A8
- net A8: now also J1.25 (A8); no longer U1.1 (B8/TDI)
- net D1 renamed D1/TMS
- net D1/TMS: now also U1.7 (D0/TMS), J1.12 (D1); no longer U1.25 (C1)
- net D2: no longer names the net of U1.27 (A14)
- net D2: no longer U2.33 (DQ2)
- net D3 renamed D3/TDO
- net D3/TDO: now also U1.32 (A8/TDO), J1.15 (D3); no longer U1.28 (A13)
- net D5/TDO renamed D5/TCK
- net D5/TCK: now also U1.26 (C0/TCK), J1.17 (D5); no longer U1.32 (A8/TDO)
- net ~{CE} renamed ~{SRAM_CE}
- net ~{SRAM_CE}: now also U1.21 (C9); no longer U1.10 (D3)
- net ~{OE} renamed ~{SRAM_OE}
- net ~{SRAM_OE}: now also U1.20 (C10); no longer U1.8 (D1)
- net ~{WE} renamed ~{SRAM_WE}
- net ~{SRAM_WE}: now also U1.18 (C12); no longer U1.30 (A10)
- new net D2/TDI: J1.13 (D2), U1.1 (B8/TDI), U2.33 (DQ2)
- no-connect marks 11 -> 9
Other:
- note added: "29F800 bottom-boot TSOP-48 AM29F800BB MX29F800CB M29F800FB"
- note added: "NOTICE: This is only an alternative PCB for DIP REX# (REX# for NEC PC-8201/8300 or Olivetti M10). The bitstream to program the CPLD is not publicly available."
- note removed: "29F800 bottom-boot TSOP-48 AM29F800BB, MX29F800CB, M29F800FB"
- note removed: "BRIDGE ["
- note removed: "CPLD Programming"
- note removed: "GND"
- note removed: "POWER IN ["
- note removed: "Steve Adolph has not published either the HDL source nor bitstream to program the CPLD for REX Classic NEC, and it is not the same as for REX Classic for Model 100/200. To use this pcb you can do one of the following: * Dump the .jed from another REX Classic NEC * Desolder and transplant the CPLD chip from another REX Classic NEC * Write new HDL"
- note removed: "TCK"
- note removed: "TDI"
- note removed: "TDO"
- note removed: "TMS"
- note removed: "VREF"
- note removed: "XCR3032XL or XCR3064XL"
- note removed: "~{RESET}"
- title: REX Classic NEC bkw -> REX Sharp DIP bkw
- moved on the sheet: C1, R1, U3
