File: REX_Sharp_DIP_bkw.kicad_pcb (KiCad board)
At the start: 2 copper layers, 35.6 x 17.8 mm, 10 parts, among them J1 Option-ROM SOCKET, U1 XCR3032XL-VQ44, U2 29F800 bottom boot, U3 LP2980-3.3

Commit message: silkscreen
Parts:
- U2: value 29F800 bottom boot -> 29F800BB
- moved U3 0.32 mm to (156.2, 98.5)
Routing:
- net +5V: track 37.4 -> 36.6 mm
