File: REXCPM_bkw.kicad_sch (KiCad schematic)
At the start: 18 parts, among them J1 Tandy_100_102_200_option_rom, J2 Conn_01x03_Pin, U1 XCR3064XL, U2 CY61277, U3 4245, U4 4245, U5 NCV563SQ33, U6 NCV563SQ33

Commit message: rexcpm small layout opts
Parts:
- U2: value CY61277 -> RMLV3216AGSA
Other:
- note added: "To program the CPLD Solder a piece of wire to JP1 with one end of the wire bridging JP1 and the other end free. Insert a Molex 78805 socket (15-29-9282) in a breadboard. Connect socket DIP pins pin 1 - power 5v pin 12 - jtag TMS pin 13 - jtag TDI pin 14 - power GND, jtag GND pin 15 - jtag TDO pin 17 - jtag TCK Insert REXCPM in socket. Connect jtag VREF (VCC/3v3) to wire on JP1 After programming, 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"
Changed lines of the file:
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@@
   (title_block
     (title "REXCPM bkw")
-    (date "2023-10-07")
-    (rev "003")
+    (date "2023-11-05")
+    (rev "005")
     (company "Brian K. White - b.kenyon.w@gmail.com")
     (comment 1 "Original design: Steven Adolph")
@@
   (wire (pts (xy 322.58 139.7) (xy 325.12 139.7))
     (stroke (width 0) (type default))
+  )
+  (text "To program the CPLD\n\nSolder a piece of wire to JP1 with one end of the wire bridging JP1 and the other end free.\n\nInsert a Molex 78805 socket (15-29-9282) in a breadboard.\n\nConnect socket DIP pins\npin  1 - power 5v\npin 12 - jtag TMS\npin 13 - jtag TDI\npin 14 - power GND, jtag GND\npin 15 - jtag TDO\npin 17 - jtag TCK\n\nInsert REXCPM in socket.\n\nConnect jtag VREF (VCC/3v3) to wire on JP1\n\nAfter programming, desolder wire from JP1 and leave JP1 open."
+    (at 25.4 266.7 0)
+    (effects (font (size 1.27 1.27)) (justify left bottom))
   )
   (text "74LVC4245APW_118" (at 231.14 57.15 0)
@@
       (effects (font (size 1.524 1.524)) (justify left))
     )
-    (property "Value" "CY61277" (at 326.0441 66.04 0)
+    (property "Value" "RMLV3216AGSA" (at 326.0441 66.04 0)
       (effects (font (size 1.524 1.524)) (justify left))
     )
@@
       (effects (font (size 1.524 1.524)) hide)
     )
-    (property "Datasheet" "datasheets/CY62177EV30LL.pdf" (at 323.85 101.6 0)
+    (property "Datasheet" "datasheets/RMLV3216AGSA.pdf" (at 323.85 101.6 0)
       (effects (font (size 1.524 1.524)) hide)
     )

Commit message: rexcpm qwiic connector
Parts:
- J2: value Conn_01x03_Pin -> SM04B; footprint 000_LOCAL:PinHeader_1x04_P2.54mm_Horizontal -> 000_LOCAL:JST_SH_SM04B-SRSS-TB_1x04-1MP_P1.00mm_Horizontal; symbol 000_LOCAL:Conn_01x04_Pin -> 000_LOCAL:Conn_01x04_MountingPin
Connections:
- net GND: now also J2.MP (MountPin)
- net RAM_RST: now also J2.4 (Pin_4); no longer J2.2 (Pin_2)
- net ~{BUS_WR}: now also J2.2 (Pin_2); no longer J2.4 (Pin_4)
Other:
- note added: "To REXCPM_UPS"
- note removed: "System Bus Interface / REXCPM_UPS"
Changed lines of the file:
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@@
   (title_block
     (title "REXCPM bkw")
-    (date "2023-11-05")
-    (rev "005")
+    (date "2023-11-06")
+    (rev "006")
     (company "Brian K. White - b.kenyon.w@gmail.com")
     (comment 1 "Original design: Steven Adolph")
@@
     (stroke (width 0) (type default))
   )
-  (wire (pts (xy 78.74 172.72) (xy 203.2 172.72))
-    (stroke (width 0) (type default))
-  )
   (wire (pts (xy 133.35 170.18) (xy 133.35 124.46))
     (stroke (width 0) (type default))
@@
     (stroke (width 0) (type default))
   )
+  (wire (pts (xy 133.35 172.72) (xy 78.74 172.72))
+    (stroke (width 0) (type default))
+  )
   (wire (pts (xy 60.96 147.32) (xy 135.89 147.32))
     (stroke (width 0) (type default))
@@
     (stroke (width 0) (type default))
   )
-  (wire (pts (xy 114.3 167.64) (xy 114.3 203.2))
-    (stroke (width 0) (type default))
-  )
-  (wire (pts (xy 78.74 167.64) (xy 114.3 167.64))
+  (wire (pts (xy 133.35 172.72) (xy 133.35 203.2))
     (stroke (width 0) (type default))
   )
@@
     (stroke (width 0) (type default))
   )
-  (wire (pts (xy 203.2 172.72) (xy 203.2 152.4))
-    (stroke (width 0) (type default))
-  )
   (wire (pts (xy 238.76 104.14) (xy 226.06 104.14))
     (stroke (width 0) (type default))
@@
     (stroke (width 0) (type default))
   )
+  (wire (pts (xy 78.74 167.64) (xy 203.2 167.64))
+    (stroke (width 0) (type default))
+  )
   (wire (pts (xy 67.31 116.84) (xy 76.2 116.84))
     (stroke (width 0) (type default))
@@
     (stroke (width 0) (type default))
   )
-  (wire (pts (xy 114.3 203.2) (xy 144.78 203.2))
+  (wire (pts (xy 133.35 203.2) (xy 144.78 203.2))
     (stroke (width 0) (type default))
   )
@@
   )
   (wire (pts (xy 341.63 152.4) (xy 341.63 132.08))
+    (stroke (width 0) (type default))
+  )
+  (wire (pts (xy 203.2 167.64) (xy 203.2 152.4))
     (stroke (width 0) (type default))
   )
@@
     (effects (font (size 1.27 1.27)) (justify left bottom))
   )
-  (text "System Bus Interface / REXCPM_UPS" (at 57.15 157.48 0)
+  (text "To REXCPM_UPS" (at 64.77 157.48 0)
     (effects (font (size 1.27 1.27)) (justify left bottom))
   )
@@
     (effects (font (size 1.27 1.27)) (justify left bottom))
   )
-  (label "RAM" (at 80.01 170.18 0) (fields_autoplaced)
+  (label "RAM" (at 78.74 170.18 0) (fields_autoplaced)
     (effects (font (size 1.27 1.27)) (justify left bottom))
   )
@@
     (effects (font (size 1.27 1.27)) (justify right bottom))
   )
-  (label "RAM_RST" (at 80.01 167.64 0) (fields_autoplaced)
+  (label "RAM_RST" (at 78.74 172.72 0) (fields_autoplaced)
     (effects (font (size 1.27 1.27)) (justify left bottom))
   )
@@
     (effects (font (size 1.27 1.27)) (justify left bottom))
   )
-  (label "~{BUS_WR}" (at 80.01 172.72 0) (fields_autoplaced)
+  (label "~{BUS_WR}" (at 78.74 167.64 0) (fields_autoplaced)
     (effects (font (size 1.27 1.27)) (justify left bottom))
   )
@@
         (path "/121db428-1a06-4610-a5f5-4dc5441e94b6"
           (reference "#PWR017") (unit 1)
+        )
+      )
+    )
+  )
+  (symbol (lib_id "power:GND") (at 73.66 177.8 0) (unit 1)
+    (in_bom yes) (on_board yes) (dnp no)
+    (property "Reference" "#PWR01" (at 73.66 184.15 0)
+      (effects (font (size 1.27 1.27)) hide)
+    )
+    (property "Value" "GND" (at 73.66 181.61 0)
+      (effects (font (size 1.27 1.27)))
+    )
+    (property "Footprint" "" (at 73.66 177.8 0)
+      (effects (font (size 1.27 1.27)) hide)
+    )
+    (property "Datasheet" "" (at 73.66 177.8 0)
+      (effects (font (size 1.27 1.27)) hide)
+    )
+    (pin "1")
+    (instances
+      (project "REXCPM_bkw"
+        (path "/121db428-1a06-4610-a5f5-4dc5441e94b6"
+          (reference "#PWR01") (unit 1)
         )
       )
@@
     )
   )
-  (symbol (lib_id "000_LOCAL:Conn_01x04_Pin") (at 73.66 167.64 0) (unit 1)
+  (symbol (lib_id "000_LOCAL:Conn_01x04_MountingPin") (at 73.66 167.64 0) (mirror y) (unit 1)
     (in_bom yes) (on_board yes) (dnp no)
     (property "Reference" "J2" (at 73.66 158.75 0)
       (effects (font (size 1.27 1.27)))
     )
-    (property "Value" "Conn_01x03_Pin" (at 73.66 161.29 0)
-      (effects (font (size 1.27 1.27)))
-    )
-    (property "Footprint" "000_LOCAL:PinHeader_1x04_P2.54mm_Horizontal" (at 73.66 167.64 0)
-      (effects (font (size 1.27 1.27)) hide)
-    )
-    (property "Datasheet" "~" (at 73.66 167.64 0)
+    (property "Value" "SM04B" (at 73.66 161.29 0)
+      (effects (font (size 1.27 1.27)))
+    )
+    (property "Footprint" "000_LOCAL:JST_SH_SM04B-SRSS-TB_1x04-1MP_P1.00mm_Horizontal" (at 73.66 167.64 0)
+      (effects (font (size 1.27 1.27)) hide)
+    )
+    (property "Datasheet" "datasheets/eSH.pdf" (at 73.66 167.64 0)
       (effects (font (size 1.27 1.27)) hide)
     )
@@
     (pin "3")
     (pin "4")
-    (instances
-      (project "REXCPM_bkw"
+    (pin "MP")
+    (instances
+      (project "REXCPM_bkw"

Commit message: rexcpm add cap on vbus
Parts:
- added C6: 4.7u, 000_LOCAL:C_0805, symbol 000_LOCAL:C
Connections:
- net GND: now also C6.2
- net VBUS: now also C6.1
Changed lines of the file:
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@@
     (title "REXCPM bkw")
     (date "2023-11-06")
-    (rev "006")
+    (rev "007")
     (company "Brian K. White - b.kenyon.w@gmail.com")
     (comment 1 "Original design: Steven Adolph")
@@
     )
   )
+  (symbol (lib_id "000_LOCAL:C") (at 177.8 207.01 0) (unit 1)
+    (in_bom yes) (on_board yes) (dnp no)
+    (property "Reference" "C6" (at 175.26 205.74 0)
+      (effects (font (size 1.4986 1.4986)) (justify right))
+    )
+    (property "Value" "4.7u" (at 175.26 208.28 0)
+      (effects (font (size 1.4986 1.4986)) (justify right))
+    )
+    (property "Footprint" "000_LOCAL:C_0805" (at 177.8 207.01 0)
+      (effects (font (size 1.27 1.27)) hide)
+    )
+    (property "Datasheet" "" (at 177.8 207.01 0)
+      (effects (font (size 1.27 1.27)) hide)
+    )
+    (pin "1")
+    (pin "2")
+    (instances
+      (project "REXCPM_bkw"
+        (path "/121db428-1a06-4610-a5f5-4dc5441e94b6"
+          (reference "C6") (unit 1)
+        )
+      )
+    )
+  )
   (symbol (lib_id "power:GND") (at 190.5 240.03 0) (unit 1)
     (in_bom yes) (on_board yes) (dnp no)
@@
         )
       )
+    )
+  )
+  (symbol (lib_id "power:GND") (at 177.8 210.82 0) (unit 1)
+    (in_bom yes) (on_board yes) (dnp no)
+    (property "Reference" "#PWR030" (at 177.8 217.17 0)
+      (effects (font (size 1.27 1.27)) hide)
+    )
+    (property "Value" "GND" (at 177.8 214.63 0)
+      (effects (font (size 1.27 1.27)))
+    )
+    (property "Footprint" "" (at 177.8 210.82 0)
+      (effects (font (size 1.27 1.27)) hide)
+    )
+    (property "Datasheet" "" (at 177.8 210.82 0)
+      (effects (font (size 1.27 1.27)) hide)
+    )
+    (pin "1")
+    (instances
+      (project "REXCPM_bkw"
+        (path "/121db428-1a06-4610-a5f5-4dc5441e94b6"
+          (reference "#PWR030") (unit 1)
+        )
+      )
