File: PCB/REXCPM_bkw.kicad_pcb (KiCad board)
At the start: 2 copper layers, 38 x 16.6 mm, 19 parts, among them J1 Tandy_100_102_200_option_rom, J2 SM04B, U1 XCR3064XL, U2 RMLV3216AGSA, U3 4245, U4 4245, U5 NCV563SQ33, U6 NCV563SQ33

Commit message: silkscreen
Other:
- board text added: "CY61277EV30LL AS6C3216A-55TIN"
Changed lines of the file:
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@@
     (effects (font (size 0.8 0.8) (thickness 0.15) bold) (justify mirror))
+  )
+  (gr_text "CY61277EV30LL\nAS6C3216A-55TIN" (at 129.8884 98.087 180) (layer "B.SilkS")
+    (effects (font (size 0.8 0.8) (thickness 0.1)) (justify top mirror))
   )
   (gr_text "TCK" (at 148.623 92.1766) (layer "B.SilkS")
