File: PCB/REXCPM_bkw.kicad_sch (KiCad schematic)
At the start: 19 parts, among them J1 Tandy_100_102_200_option_rom, J2 SM04B, U1 XCR3064XL, U2 RMLV3216AGSA, U3 4245, U4 4245, U5 NCV563SQ33, U6 NCV563SQ33

Commit message: silkscreen
Connections:
- net +VSW renamed Vall
Changed lines of the file:
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@@
   (junction (at 167.64 66.04) (diameter 0) (color 0 0 0 0)
   )
+  (junction (at 165.1 208.28) (diameter 0) (color 0 0 0 0)
+  )
   (junction (at 341.63 104.14) (diameter 0) (color 0 0 0 0)
   )
@@
   )
   (junction (at 341.63 101.6) (diameter 0) (color 0 0 0 0)
-  )
-  (junction (at 177.8 229.87) (diameter 0) (color 0 0 0 0)
   )
   (no_connect (at 306.07 127))
@@
     (stroke (width 0) (type default))
   )
-  (wire (pts (xy 177.8 229.87) (xy 182.88 229.87))
-    (stroke (width 0) (type default))
-  )
   (wire (pts (xy 341.63 104.14) (xy 341.63 106.68))
     (stroke (width 0) (type default))
@@
     (stroke (width 0) (type default))
   )
-  (wire (pts (xy 165.1 229.87) (xy 177.8 229.87))
+  (wire (pts (xy 165.1 229.87) (xy 182.88 229.87))
     (stroke (width 0) (type default))
   )
@@
   (label "SRAM_A1" (at 256.54 83.82 0) (fields_autoplaced)
     (effects (font (size 1.27 1.27)) (justify left bottom))
+  )
+  (label "Vall" (at 162.56 208.28 180) (fields_autoplaced)
+    (effects (font (size 1.27 1.27)) (justify right bottom))
   )
   (label "SRAM_A14" (at 306.07 106.68 180) (fields_autoplaced)
@@
     )
   )
+  (symbol (lib_id "power:PWR_FLAG") (at 165.1 208.28 0) (unit 1)
+    (in_bom yes) (on_board yes) (dnp no)
+    (property "Reference" "#FLG01" (at 165.1 206.375 0)
+      (effects (font (size 1.27 1.27)) hide)
+    )
+    (property "Value" "PWR_FLAG" (at 165.1 204.47 0)
+      (effects (font (size 1.27 1.27)) hide)
+    )
+    (property "Footprint" "" (at 165.1 208.28 0)
+      (effects (font (size 1.27 1.27)) hide)
+    )
+    (property "Datasheet" "~" (at 165.1 208.28 0)
+      (effects (font (size 1.27 1.27)) hide)
+    )
+    (pin "1")
+    (instances
+      (project "REXCPM_bkw"
+        (path "/121db428-1a06-4610-a5f5-4dc5441e94b6"
+          (reference "#FLG01") (unit 1)
+        )
+      )
+    )
+  )
   (symbol (lib_id "power:GND") (at 190.5 240.03 0) (unit 1)
     (in_bom yes) (on_board yes) (dnp no)
@@
         )
       )
-    )
-  )
-  (symbol (lib_id "power:+VSW") (at 177.8 229.87 0) (unit 1)
-    (in_bom yes) (on_board yes) (dnp no)
-    (property "Reference" "#PWR012" (at 177.8 233.68 0)
-      (effects (font (size 1.27 1.27)) hide)
-    )
-    (property "Value" "+VSW" (at 177.8 226.06 0)
-      (effects (font (size 1.27 1.27)))
-    )
-    (property "Footprint" "" (at 177.8 229.87 0)
-      (effects (font (size 1.27 1.27)) hide)
-    )
-    (property "Datasheet" "" (at 177.8 229.87 0)
-      (effects (font (size 1.27 1.27)) hide)
-    )
-    (pin "1")
-    (instances
-      (project "REXCPM_bkw"
-        (path "/121db428-1a06-4610-a5f5-4dc5441e94b6"
-          (reference "#PWR012") (unit 1)
-        )
-      )
