File: PCB/REX_Sharp_JEDEC_bkw.kicad_pcb (KiCad board)
At the start: 2 copper layers, 35.6 x 17.8 mm, 10 parts, among them J1 Option-ROM SOCKET, U1 XCR3032XL-VQ44, U2 29F800BB, U3 LP2980-3.3

Commit message: add sharp-tandy
Changed lines of the file:
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@@
 	(paper "A4")
 	(title_block
-		(title "REX_Sharp_DIP_bkw")
+		(title "REX_Sharp_JEDEC_bkw")
 		(date "2023-07-04")
 		(rev "008")
@@
 				(font
 					(size 1.27 1.27)
+					(thickness 0.15)
 				)
 			)
@@
 				(font
 					(size 1.27 1.27)
+					(thickness 0.15)
 				)
 			)
@@
 				(font
 					(size 1.27 1.27)
+					(thickness 0.15)
 				)
 			)
@@
 				(font
 					(size 1.27 1.27)
+					(thickness 0.15)
 				)
 			)
@@
 				(font
 					(size 1.27 1.27)
+					(thickness 0.15)
 				)
 			)
@@
 				(font
 					(size 1.27 1.27)
+					(thickness 0.15)
 				)
 			)
@@
 				(font
 					(size 1.27 1.27)
+					(thickness 0.15)
 				)
 			)
@@
 				(font
 					(size 1.27 1.27)
+					(thickness 0.15)
 				)
 			)
@@
 				(font
 					(size 1.27 1.27)
+					(thickness 0.15)
 				)
 			)
@@
 				(font
 					(size 1.27 1.27)
+					(thickness 0.15)
 				)
 			)
@@
 				(font
 					(size 1.27 1.27)
+					(thickness 0.15)
 				)
 			)
@@
 				(font
 					(size 1.27 1.27)
+					(thickness 0.15)
 				)
 			)
@@
 				(font
 					(size 1.27 1.27)
+					(thickness 0.15)
 				)
 			)
@@
 				(font
 					(size 1.27 1.27)
+					(thickness 0.15)
 				)
 			)
@@
 				(font
 					(size 1.27 1.27)
+					(thickness 0.15)
 				)
 			)
@@
 				(font
 					(size 1.27 1.27)
+					(thickness 0.15)
 				)
 			)
@@
 				(font
 					(size 1.27 1.27)
+					(thickness 0.15)
 				)
 			)
@@
 				(font
 					(size 1.27 1.27)
+					(thickness 0.15)
 				)
 			)
@@
 				(font
 					(size 1.27 1.27)
+					(thickness 0.15)
 				)
 			)
@@
 				(font
 					(size 1.27 1.27)
+					(thickness 0.15)
 				)
 			)
@@
 				(font
 					(size 1.27 1.27)
+					(thickness 0.15)
 				)
 			)
@@
 				(font
 					(size 1.27 1.27)
+					(thickness 0.15)
 				)
 			)
@@
 				(font
 					(size 1.27 1.27)
+					(thickness 0.15)
 				)
 			)
@@
 				(font
 					(size 1.27 1.27)
+					(thickness 0.15)
 				)
 			)
@@
 				(font
 					(size 1.27 1.27)
+					(thickness 0.15)
 				)
 			)
@@
 				(font
 					(size 1.27 1.27)
+					(thickness 0.15)
 				)
 			)
@@
 				(font
 					(size 1.27 1.27)
+					(thickness 0.15)
 				)
 			)
@@
 				(font
 					(size 1.27 1.27)
+					(thickness 0.15)
 				)
 			)
@@
 				(font
 					(size 1.27 1.27)
+					(thickness 0.15)
 				)
 			)
@@
 				(font
 					(size 1.27 1.27)
+					(thickness 0.15)
 				)
 			)
