File: PCB/REX_Sharp_TANDY_bkw.kicad_sch (KiCad schematic)
At the start: 10 parts, among them J1 Option-ROM SOCKET, U1 XCR3032XL-VQ44, U2 29F800 bottom boot, U3 LP2980-3.3

Commit message: add sharp-tandy
Parts:
- removed J1: Option-ROM SOCKET, 000_LOCAL:DIP-28_600_pcb_shallow_notch, symbol 000_LOCAL:ROM_SOCKET
- added J1: ROM_SOCKET_TANDY, 000_LOCAL:Molex78802_PCB_28, symbol 000_LOCAL:ROM_SOCKET_TANDY
- C1, C3: value 1uF -> 1u
- C2: value 100pF -> 100p
Connections:
- net +5V: now also J1.1 (VCC)
- net A0: now also J1.10 (A0)
- net A1: now also J1.9 (A1)
- net A10: now also U2.18 (A7), J1.2 (A10); no longer U2.7 (A9)
- net A11: now also U2.3 (A13), J1.20 (A11); no longer U2.6 (A10)
- net A12: now also J1.24 (A12)
- net A13: now also J1.22 (A13)
- net A14: now also U2.48 (A16), J1.28 (A14); no longer U2.3 (A13)
- net A17: now also U2.6 (A10); no longer U2.48 (A16)
- net A2: now also J1.8 (A2)
- net A3: now also J1.7 (A3)
- net A4: now also J1.6 (A4)
- net A5: now also J1.5 (A5)
- net A6: now also J1.4 (A6)
- net A7: now also J1.3 (A7)
- net A8: now also U2.8 (A8), J1.26 (A8); no longer U2.18 (A7)
- net A9: now also U2.7 (A9), J1.25 (A9); no longer U2.8 (A8)
- net D0: now also J1.11 (AD0)
- net D1/TMS: now also J1.12 (AD1)
- net D2/TDI: now also J1.13 (AD2)
- net D3/TDO: now also J1.15 (AD3)
- net D4: now also J1.16 (AD4)
- net D5/TCK: now also J1.17 (AD5)
- net D6: now also J1.18 (AD6)
- net D7: now also J1.19 (AD7)
- net GND: now also J1.14 (GND)
- net ~{BUS_CS}: now also J1.27 (~{CS})
- net ~{BUS_OE}: now also J1.21 (~{OE})
- no-connect marks 9 -> 10
Other:
- note added: "NOTICE: This is only an alternative PCB for REX# for TANDY 100, 102, 200. The bitstream to program the CPLD is not publicly available."
- note removed: "NOTICE: This is only an alternative PCB for DIP REX# (REX# for NEC PC-8201/8300 or Olivetti M10). The bitstream to program the CPLD is not publicly available."
- title: REX Sharp DIP bkw -> REX Sharp TANDY bkw
- moved on the sheet: C1, C3, R1, U3
