File: PCB/REX_Classic_bkw.kicad_pcb (KiCad board)
At the start: 2 copper layers, 38 x 16.6 mm, 12 parts, among them J1 Tandy_100_102_200_option_rom, J2 JTAG, J3 PRG, U1 XCR3064XL-VQ44, U2 29F800BB, U3 LP2980-3.3

Commit message: remove dead shapeways url for carrier
Other:
- board text added: "R*: ${00000000-0000-0000-0000-00005d099a58:VALUE} C*: ${00000000-0000-0000-0000-00005d17005c:VALUE} U3: ${00000000-0000-0000-0000-00005e3c09df:VALUE}"
- board text removed: "R*: ${00000000-0000-0000-0000-00005d099a58:VALUE} C*: ${00000000-0000-0000-0000-00005d17005c:VALUE} U3: ${00000000-0000-0000-0000-00005e3c09df:VALUE} shpws.me/SGGB"
