File: PCB/REX_Classic_bkw.kicad_sch (KiCad schematic)
At the start: 12 parts, among them J1 Tandy_100_102_200_option_rom, J2 JTAG, J3 PRG, U1 XCR3064XL-VQ44, U2 29F800BB, U3 LP2980-3.3

Commit message: remove dead shapeways url for carrier
Parts:
- C1, C2, C3: value 1uF -> 1u
Other:
- moved on the sheet: R1
