File: PCB/REX_Classic_bkw.kicad_sch (KiCad schematic)
At the start: 12 parts, among them J1 Tandy_100_102_200_option_rom, J2 JTAG, J3 PRG, U1 XCR3064XL-VQ44, U2 29F800BB, U3 LP2980-3.3

Commit message: housing component, fillet tracks, molex datasheets corrections
Parts:
- added N1: Molex78802_PCB_28 Carrier, 000_LOCAL:Housing_Molex78802_PCB_28, symbol 000_LOCAL:Housing
- U1: MPN (none) -> XCR3064XL-VQ44
- U2: MPN (none) -> AM29F800BB
- U3: MPN (none) -> LP2980-3.3
Other:
- moved on the sheet: R1
